Commit message: Add simple Azure Kinect URDF

File: urdf/azure_kinect.urdf (robot description, URDF)
Before this commit: robot azure-kinect, 2 links, 1 joints
Links:
- added link camera_visor; visual box size=0.026 0.101 0.037
Joints:
- added joint camera_base_to_visor: type fixed, parent camera_base, child camera_visor, origin xyz=0. 0. 0. rpy=0. 0. 0.
