Commit message: Use xacro to generate urdf model with tf_prefix

File: urdf/azure_kinect.urdf.xacro (robot description, xacro)
@@ -4,5 +4,6 @@
  Licensed under the MIT License.
  -->
-<robot name="azure-kinect">
+<robot name="azure-kinect" xmlns:xacro="http://www.ros.org/wiki/xacro">
+  <xacro:arg name="tf_prefix" default=""/>
   <material name="black">
     <color rgba="0. 0. 0. 1" />
@@ -17,5 +18,5 @@
     <color rgba="0.9 0.9 0.9 1" />
   </material>
-  <link name="camera_body">
+  <link name="$(arg tf_prefix)camera_body">
     <visual>
       <origin xyz="0. 0. 0." />
@@ -26,5 +27,5 @@
     </visual>
   </link>
-  <link name="camera_base">
+  <link name="$(arg tf_prefix)camera_base">
     <visual>
       <origin xyz="-0.013 0. 0." />
@@ -35,5 +36,5 @@
     </visual>
   </link>
-  <link name="camera_visor">
+  <link name="$(arg tf_prefix)camera_visor">
     <visual>
       <origin xyz="-0.0128 0. 0." />
@@ -44,12 +45,12 @@
     </visual>
   </link>
-  <joint name="camera_base_to_body" type="fixed">
-    <parent link="camera_base" />
-    <child link="camera_body" />
+  <joint name="$(arg tf_prefix)camera_base_to_body" type="fixed">
+    <parent link="$(arg tf_prefix)camera_base" />
+    <child link="$(arg tf_prefix)camera_body" />
     <origin xyz="-0.0757 0. 0.008" rpy="0. 0. 0." />
   </joint>
-  <joint name="camera_base_to_visor" type="fixed">
-    <parent link="camera_base" />
-    <child link="camera_visor" />
+  <joint name="$(arg tf_prefix)camera_base_to_visor" type="fixed">
+    <parent link="$(arg tf_prefix)camera_base" />
+    <child link="$(arg tf_prefix)camera_visor" />
     <origin xyz="0. 0. 0." rpy="0. 0. 0." />
   </joint>

Commit message: Added in xacro file processing and removed arg

File: urdf/azure_kinect.urdf.xacro (robot description, xacro)
@@ -5,5 +5,4 @@
  -->
 <robot name="azure-kinect" xmlns:xacro="http://www.ros.org/wiki/xacro">
-  <xacro:arg name="tf_prefix" default=""/>
   <material name="black">
     <color rgba="0. 0. 0. 1" />
@@ -18,5 +17,5 @@
     <color rgba="0.9 0.9 0.9 1" />
   </material>
-  <link name="$(arg tf_prefix)camera_body">
+  <link name="camera_body">
     <visual>
       <origin xyz="0. 0. 0." />
@@ -27,5 +26,5 @@
     </visual>
   </link>
-  <link name="$(arg tf_prefix)camera_base">
+  <link name="camera_base">
     <visual>
       <origin xyz="-0.013 0. 0." />
@@ -36,5 +35,5 @@
     </visual>
   </link>
-  <link name="$(arg tf_prefix)camera_visor">
+  <link name="camera_visor">
     <visual>
       <origin xyz="-0.0128 0. 0." />
@@ -45,12 +44,12 @@
     </visual>
   </link>
-  <joint name="$(arg tf_prefix)camera_base_to_body" type="fixed">
-    <parent link="$(arg tf_prefix)camera_base" />
-    <child link="$(arg tf_prefix)camera_body" />
+  <joint name="camera_base_to_body" type="fixed">
+    <parent link="camera_base" />
+    <child link="camera_body" />
     <origin xyz="-0.0757 0. 0.008" rpy="0. 0. 0." />
   </joint>
-  <joint name="$(arg tf_prefix)camera_base_to_visor" type="fixed">
-    <parent link="$(arg tf_prefix)camera_base" />
-    <child link="$(arg tf_prefix)camera_visor" />
+  <joint name="camera_base_to_visor" type="fixed">
+    <parent link="camera_base" />
+    <child link="camera_visor" />
     <origin xyz="0. 0. 0." rpy="0. 0. 0." />
   </joint>
