Commit message: corrected tilt angle of depth frame and added 'camera_base' frame for compatability

File: urdf/azure_kinect_macro.urdf.xacro (robot description, xacro)
@@ -27,7 +27,13 @@
       </collision>
     </link>
+    <link name="${prefix}camera_base" /> <!-- for compatability with old model -->
     <link name="${prefix}azure_rgb" />
     <link name="${prefix}azure_depth" />
     <link name="${prefix}azure_gyro" />
+    <joint name="${prefix}azure_base_to_camera_base" type="fixed">
+      <parent link="${prefix}azure_base" />
+      <child link="${prefix}camera_base" />
+      <origin xyz="0.062 0.0 0.0065" rpy="0 0 0" />
+    </joint>
     <joint name="${prefix}azure_base_to_rgb" type="fixed">
       <parent link="${prefix}azure_base" />
@@ -38,5 +44,5 @@
       <parent link="${prefix}azure_base" />
       <child link="${prefix}azure_depth" />
-      <origin xyz="0.0618 -0.0005 0.0065" rpy="-${pi/2} 0 -${pi/2}" />
+      <origin xyz="0.0618 -0.0005 0.0065" rpy="-${96/180*pi} 0 -${pi/2}" />
     </joint>
     <joint name="${prefix}azure_base_to_gyro" type="fixed">

Commit message: tilted gazebo frame as well

File: urdf/azure_kinect_macro.urdf.xacro (robot description, xacro)
@@ -55,8 +55,8 @@
            (see #243 https://github.com/ros-simulation/gazebo_ros_pkgs/issues/243) -->
       <link name="${prefix}azure_gazebo_depth" />
-      <joint name="${prefix}azure_depth_to_gazebo_depth" type="fixed">
+      <joint name="${prefix}azure_base_to_gazebo_depth" type="fixed">
         <parent link="${prefix}azure_base" />
         <child link="${prefix}azure_gazebo_depth"/>
-        <origin xyz="0.0618 -0.0005 0.0065" rpy="0 0 0"/>
+        <origin xyz="0.0618 -0.0005 0.0065" rpy="0 ${6/180*pi} 0"/>
       </joint>
       <gazebo reference="${prefix}azure_gazebo_depth">

Commit message: new parameter to switch between CAD data and factory calibration

File: urdf/azure_kinect_macro.urdf.xacro (robot description, xacro)
@@ -16,5 +16,5 @@
  -->
 <robot name="azure_kinect" xmlns:xacro="http://www.ros.org/wiki/xacro">
-  <xacro:macro name="azure_kinect" params="prefix:='' parent:='' gazebo:=false *origin">
+  <xacro:macro name="azure_kinect" params="prefix:='' parent:='' publish_calibrated_poses=true gazebo:=false *origin">
     <xacro:if value="${parent != ''}">
       <joint name="${prefix}azure_in_joint" type="fixed">
@@ -38,8 +38,30 @@
       </collision>
     </link>
-    <link name="${prefix}camera_base" /> <!-- for compatability with old model -->
-    <link name="${prefix}azure_rgb" />
-    <link name="${prefix}azure_depth" />
-    <link name="${prefix}azure_gyro" />
+    <link name="${prefix}azure_camera_base" /> <!-- for compatability with calibration parameters -->
+    <joint name="${prefix}azure_base_to_camera_base" type="fixed">
+      <parent link="${prefix}azure_base" />
+      <child link="${prefix}azure_camera_base" />
+      <origin xyz="0.062 0.0 0.0065" rpy="0 0 0" />
+    </joint>
+    <xacro:if value="${not publish_calibrated_poses or gazebo}">
+      <link name="${prefix}azure_rgb" />
+      <link name="${prefix}azure_depth" />
+      <link name="${prefix}azure_imu" />
+      <joint name="${prefix}azure_base_to_rgb" type="fixed">
+        <parent link="${prefix}azure_base" />
+        <child link="${prefix}azure_rgb" />
+        <origin xyz="0.0618 -0.032 0.0065" rpy="-${pi/2} 0 -${pi/2}" />
+      </joint>
+      <joint name="${prefix}azure_base_to_depth" type="fixed">
+        <parent link="${prefix}azure_base" />
+        <child link="${prefix}azure_depth" />
+        <origin xyz="0.0618 -0.0005 0.0065" rpy="-${96/180*pi} 0 -${pi/2}" />
+      </joint>
+      <joint name="${prefix}azure_base_to_imu" type="fixed">
+        <parent link="${prefix}azure_base" />
+        <child link="${prefix}azure_imu" />
+        <origin xyz="0.0618 -0.0005 0.0065" rpy="0 ${pi} 0" />
+      </joint>
+    </xacro:if>
     <link name="${prefix}azure_microphone_0" />
     <link name="${prefix}azure_microphone_1" />
@@ -49,24 +71,4 @@
     <link name="${prefix}azure_microphone_5" />
     <link name="${prefix}azure_microphone_6" />
-    <joint name="${prefix}azure_base_to_camera_base" type="fixed">
-      <parent link="${prefix}azure_base" />
-      <child link="${prefix}camera_base" />
-      <origin xyz="0.062 0.0 0.0065" rpy="0 0 0" />
-    </joint>
-    <joint name="${prefix}azure_base_to_rgb" type="fixed">
-      <parent link="${prefix}azure_base" />
-      <child link="${prefix}azure_rgb" />
-      <origin xyz="0.0618 -0.032 0.0065" rpy="-${pi/2} 0 -${pi/2}" />
-    </joint>
-    <joint name="${prefix}azure_base_to_depth" type="fixed">
-      <parent link="${prefix}azure_base" />
-      <child link="${prefix}azure_depth" />
-      <origin xyz="0.0618 -0.0005 0.0065" rpy="-${96/180*pi} 0 -${pi/2}" />
-    </joint>
-    <joint name="${prefix}azure_base_to_gyro" type="fixed">
-      <parent link="${prefix}azure_base" />
-      <child link="${prefix}azure_gyro" />
-      <origin xyz="0.0618 -0.0005 0.0065" rpy="0 ${pi} 0" />
-    </joint>
     <joint name="${prefix}azure_base_to_microphone_0" type="fixed">
       <parent link="${prefix}azure_base" />
@@ -120,5 +122,5 @@
             WFOV 2x2 binned:      0, 5, 15, 30 FPS
             WFOV unbinned:        0, 5, 15 FPS
-            Note: Frame rate also needs to be changed in gazebo plugin settings (line 130)
+            Note: Frame rate also needs to be changed in gazebo plugin settings (line 183)
           -->
           <update_rate>5</update_rate>
@@ -146,5 +148,5 @@
                 WFOV 2x2 binned:       0.25 - 2.88 m
                 WFOV unbinned:         0.25 - 2.21 m
-                Note: Range also needs to be changed in gazebo plugin settings (lines 131 and 132)
+                Note: Range also needs to be changed in gazebo plugin settings (lines 184 and 185)
               -->
               <near>0.25</near>
@@ -154,7 +156,7 @@
           <plugin filename="libgazebo_ros_openni_kinect.so" name="${prefix}azure_camera_controller">
             <alwaysOn>true</alwaysOn>
-            <updateRate>5</updateRate>
-            <pointCloudCutoff>0.25</pointCloudCutoff>
-            <pointcloudcutoffmax>2.88</pointcloudcutoffmax>
+            <updateRate>5</updateRate> <!-- Frame rate -->
+            <pointCloudCutoff>0.25</pointCloudCutoff> <!-- Near clip distance -->
+            <pointcloudcutoffmax>2.88</pointcloudcutoffmax> <!-- Far clip distance -->
             <imageTopicName>rgb/image_raw</imageTopicName>
             <cameraInfoTopicName>rgb/camera_info</cameraInfoTopicName>

File: urdf/azure_kinect_standalone.urdf.xacro (robot description, xacro)
@@ -7,4 +7,5 @@
 <robot name="azure_kinect" xmlns:xacro="http://www.ros.org/wiki/xacro">
   <xacro:arg name="tf_prefix" default=""/>
+  <xacro:arg name="publish_calibrated_poses" default="true"/>
   <link name="$(arg tf_prefix)azure_stand">
     <visual>
@@ -22,5 +23,5 @@
   </link>
   <xacro:include filename="$(find azure_kinect_ros_driver)/urdf/azure_kinect_macro.urdf.xacro" />
-  <xacro:azure_kinect prefix="$(arg tf_prefix)" parent="$(arg tf_prefix)azure_stand" gazebo="false">
+  <xacro:azure_kinect prefix="$(arg tf_prefix)" parent="$(arg tf_prefix)azure_stand" gazebo="false" publish_calibrated_poses="$(arg publish_calibrated_poses)">
     <origin xyz="0 0 0.0235" rpy="0 -0.06 0" />
   </xacro:azure_kinect>
